File: v1/O12encoder.kicad_sch (KiCad schematic)
At the start: 16 parts, among them J1 Conn_01x06_Pin, J2 Conn_01x06_Pin, J5 JST_SM02B-SRSS-TB(LF)(SN), J6 Conn_01x06_Pin, J7 Conn_01x06_Pin, J8 Conn_01x06_Pin, U1 MA702GQ-P, U2 STM32L011F4Ux, U3 THVD1420DRLR

Commit message: readme, gen pdf
Other:
- company: (none) -> Christopher Xu
- title: (none) -> Ø12encoder
Changed lines of the file:
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@@
 (kicad_sch (version 20230121) (generator eeschema)
   (paper "A4")
+  (title_block
+    (title "Ø12encoder")
+    (date "2024-01-04")
+    (rev "1")
+    (company "Christopher Xu")
+  )
   (junction (at 133.35 151.13) (diameter 0) (color 0 0 0 0)
   )
