File: v2/O12encoder.kicad_sch (KiCad schematic)
At the start: 16 parts, among them J1 Conn_01x06_Pin, J2 Conn_01x06_Pin, J5 JST_SM02B-SRSS-TB(LF)(SN), J6 Conn_01x06_Pin, J7 Conn_01x06_Pin, J8 Conn_01x06_Pin, U1 MA702GQ-P, U2 STM32L011F4Ux, U3 THVD1420DRLR

Commit message: readme, gen pdf
Parts:
- removed J5: JST_SM02B-SRSS-TB(LF)(SN), O32controller:JST_SM02B-SRSS-TB(LF)(SN), symbol O32controller:JST_SM02B-SRSS-TB(LF)(SN)
- removed J6, J7, J8: Conn_01x06_Pin, O32controller:FFC_0.5mm_6p, symbol Connector:Conn_01x06_Pin
- removed U3: THVD1420DRLR, O32controller:THVD1420DRLR_SOT-585, symbol O32controller:THVD1420DRLR
- added D1: LED_Small, LED_SMD:LED_0603_1608Metric, symbol Device:LED_Small
- added J1 (x2): Conn_01x04, O12encoder:TE_2328702-4, symbol Connector_Generic_MountingPin:Conn_01x04_MountingPin
- added R1: R_Small_US, Resistor_SMD:R_0402_1005Metric, symbol Device:R_Small_US
- added U3: THVD1420DRLR, O12encoder:THVD1420DRLR_SOT-585, symbol O12encoder:THVD1420DRLR
- J1, J2: footprint O32controller:FFC_0.5mm_6p -> O12encoder:FFC_0.5mm_6p
- TP1, TP2, TP3, TP4: footprint O32controller:TestPoint_Pad_Rect -> O12encoder:TestPoint_Pad_Rect
- U1: footprint O32controller:MA702GQ-P -> O12encoder:MA702GQ-P; symbol O32controller:MA702GQ-P -> O12encoder:MA702GQ-P
Connections:
- net +3.3V: now also J1.1 (Pin_1), J1.1 (Pin_1), R1.1, U3.8 (VCC)
- net GND: now also J1.3 (Pin_3), J1.3 (Pin_3), J1.MP (MountPin), J1.MP (MountPin), U3.5 (GND)
- net RS485_A: now also J1.2 (Pin_2), J1.2 (Pin_2), U3.6 (A)
- net RS485_B: now also J1.4 (Pin_4), J1.4 (Pin_4), U3.7 (B)
- net UART_DE: now also U3.2 (~{RE}), U3.3 (DE)
- net UART_RX: now also U3.1 (R)
- net UART_TX: now also U3.4 (D)
- net ~{MAG2_CS}: now also U2.11 (PB1)
- net at U2.15 (PA10): now also D1.1 (K)
- new net: D1.2 (A), R1.2
- no-connect marks 15 -> 13
Other:
- note added: "GND for routing reasons set as input"
- note added: "stagger power so if connected backwards, 3.3 <-> B, GND <-> A"
- note removed: "GND for routing reasons, make sure not to GPIO output"
- note removed: "lol"
- company: (none) -> Christopher Xu
- title: (none) -> Ø12encoder: RS485 Mag Encoder
- moved on the sheet: C1, C2, C3, J1, J2, TP1, TP2, TP3, TP4, U1, U2
